File: weather_v2.0b/7seg/hardware.kicad_pcb (KiCad board)
At the start: 2 copper layers, 6 parts

Commit message: .
Parts:
- moved R2 63.8 mm to (130.0, 99.0)
- moved R1 40.5 mm to (130.0, 96.0), turned to 0 degrees
- moved DD1 29.8 mm to (104.5, 86.5)
- moved HG1 27.5 mm to (111.0, 77.0)
- moved XP1 26.5 mm to (119.5, 99.0)
- moved DD2 19.3 mm to (126.0, 85.0), turned to 0 degrees
Connections:
- DD1 pad 1: N-0000022 -> N-0000023
- DD1 pad 2: N-0000023 -> N-0000018
- DD1 pad 3: N-0000018 -> N-0000015
- DD1 pad 4: N-0000015 -> N-0000014
- DD1 pad 5: N-0000014 -> N-0000022
- HG1 pad 1: N-0000015 -> N-0000023
- HG1 pad 10: N-0000010 -> N-000006
- HG1 pad 11: N-0000011 -> N-0000012
- HG1 pad 12: N-000006 -> N-0000011
- HG1 pad 18: N-0000014 -> N-0000012
- HG1 pad 3: N-0000023 -> N-0000015
- HG1 pad 4: N-0000012 -> N-0000014
- HG1 pad 5: N-000007 -> N-000009
- HG1 pad 7: N-000005 -> N-000007
- HG1 pad 8: N-000009 -> N-000005
Routing:
- net N-000006: track 19.6 -> 77.0 mm, vias 0 -> 2
- net N-000002: track 167.9 -> 115.5 mm
- net N-0000011: track 21.3 -> 69.8 mm, vias 0 -> 2
- net /L: track 62.2 -> 27.6 mm, vias 0 -> 2
- net N-000001: track 16.8 -> 37.8 mm, vias 0 -> 2
- net N-000003: track 18.0 -> 36.8 mm, vias 0 -> 2
- net N-000007: track 21.8 -> 3.84 mm
- net N-000008: track 19.4 -> 3.96 mm
- net N-0000023: track 14.2 -> 3.53 mm
- net N-000005: track 13.4 -> 3.83 mm, vias 2 -> 0
- net N-0000010: track 8.39 -> 0.00 mm
- net N-000009: track 12.7 -> 4.43 mm
- net N-0000022: track 20.8 -> 28.4 mm, vias 2 -> 0
- net N-0000016: track 26.7 -> 19.2 mm, vias 2 -> 0
- net N-0000013: track 10.3 -> 17.5 mm
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